File: memory-300.sch (KiCad schematic (older format))
At the start: 8 parts, among them J1 Conn_02x36_Odd_Even, U1 E28F016SV, U2 TC51V16160A, U3 TC51V16160A

Commit message: Adding CERN OHL license and readme
Other:
- note added: "Copyright Randy Glenn 2018. Licensed under CERN OHL V1.2\nYou may redistribute and modify this documentation under the terms of the CERN OHL V1.2\n(http://ohwr.org/cernohl). This documentation is distributed WITHOUT ANY EXPRESS OR IMPLIED\nWARRANTY, INCLUDING MERCHANTABILITY, SATISFACTORY QUALITY AND FITNESS FOR A\nPARTICULAR PURPOSE. Please see the CERN OHL V1.2 for applicable conditions."
Changed lines of the file:
@@
 Wire Wire Line
 	5100 2400 4500 2400
+Text Notes 10450 7200 2    50   ~ 0
+Copyright Randy Glenn 2018. Licensed under CERN OHL V1.2\nYou may redistribute and modify this documentation under the terms of the CERN OHL V1.2\n(http://ohwr.org/cernohl). This documentation is distributed WITHOUT ANY EXPRESS OR IMPLIED\nWARRANTY, INCLUDING MERCHANTABILITY, SATISFACTORY QUALITY AND FITNESS FOR A\nPARTICULAR PURPOSE. Please see the CERN OHL V1.2 for applicable conditions.
 $EndSCHEMATC
